File: instrumentation_amplifier/instrumentation_amplifier.kicad_pcb (KiCad board)
At the start: 2 copper layers, 127 x 76.2 mm, 30 parts, among them CON1 1-0000001, J1 1-0000120, J2 Jumper, J3 Jumper, J4 1-0000120, SW1 1-0000852, U1 1-0000801, U2 1-0000465

Commit message: Layout Fixup
Parts:
- moved R1 55.3 mm to (106.7, 57.3)
- moved D1 55.3 mm to (110.0, 57.3)
- moved J4 1.30 mm to (164.1, 87.6), turned to 0 degrees
- moved CON1 0.89 mm to (108.3, 68.6)
Routing:
- net Net-(J4-Pad1): track 12.4 -> 13.2 mm
Other:
- board text added: "10k"
- board text added: "3-0000082 7-0000038"
- board text added: "4.5-13.2 VDC"
- board text added: "47k"
- board text added: "GND"
- board text added: "Input +"
- board text added: "Input -"
- board text added: "Instrumentation Amplifier"
- board text added: "Leeman Geophysical LLC"
- board text added: "Output"
- board text removed: "Intrumentation Amplifier"

Commit message: Switch Fixup
Parts:
- turned SW1 to 0 degrees
Routing:
- net Net-(R10-Pad1): track 15.5 -> 7.36 mm
- net Net-(R9-Pad1): track 18.5 -> 12.7 mm
- net Net-(SW1-PadC): track 11.7 -> 15.8 mm
- net Net-(R7-Pad1): track 9.46 -> 7.46 mm
