File: KiCAD_Project/instrumentation_amplifier/instrumentation_amplifier.kicad_pcb (KiCad board)
At the start: 2 copper layers, 127 x 76.2 mm, 33 parts, among them CON1 1-0000001, J1 1-0000120, J2 Jumper, J3 Jumper, J4 1-0000120, J5 NP_Conn_01x04, SW1 1-0000852, U1 1-0000801, U2 1-0000465

Commit message: Fixed jumper resistor location, silk screens, fixed J2
Parts:
- removed the G*** at (198.2, 75.3)
- moved R3 5.08 mm to (141.0, 110.5)
- moved R5 5.08 mm to (146.1, 110.5)
Connections:
- J2 pad 3: Net-(J2-Pad3) -> Net-(J1-Pad1)
- R3 pad 2: Net-(J2-Pad1) -> Net-(J2-Pad2)
- R5 pad 2: Net-(J2-Pad2) -> Net-(J2-Pad1)
- U1 pad 2: Net-(J2-Pad3) -> Net-(J1-Pad1)
- U2 pad 3: (no net) -> Net-(U2-Pad3)
- U2 pad 5: (no net) -> Net-(U2-Pad5)
Routing:
- net Net-(J1-Pad1): track 27.8 -> 43.5 mm
- net Net-(J2-Pad3): track 13.1 -> 0.00 mm

Commit message: Rev 1.1 Production
Parts:
- added G***: LOGO, lib_fp:schematic, F.Cu at (200.0, 76.7)
Connections:
- U2 pad 3: Net-(U2-Pad3) -> (no net)
- U2 pad 5: Net-(U2-Pad5) -> (no net)
Routing:
- net -5V: track 63.8 -> 74.3 mm
Other:
- board text added: "3-0000087 7-0000043"
- board text removed: "3-0000082 7-0000038"
